Commit message: first pass at changing geometry

File: src/tobor_description/urdf/tobor.xacro (robot description, xacro)
@@ -19,5 +19,5 @@
     <collision name='collision'>
       <geometry>
-        <box size=".4 .2 .1"/>
+        <box size=".78 .43 .4"/>
       </geometry>
     </collision>
@@ -25,5 +25,5 @@
       <origin xyz="0 0 0" rpy=" 0 0 0"/>
       <geometry>
-        <box size=".4 .2 .1"/>
+        <box size=".78 .43 .4"/>
       </geometry>
     </visual>
@@ -78,5 +78,5 @@
       <origin xyz="0 0 0" rpy="0 1.5707 1.5707"/>
       <geometry>
-        <cylinder radius="0.1" length="0.05"/>
+        <cylinder radius="0.15" length="0.095"/>
       </geometry>
     </collision>
@@ -84,5 +84,5 @@
       <origin xyz="0 0 0" rpy="0 1.5707 1.5707"/>
       <geometry>
-        <cylinder radius="0.1" length="0.05"/>
+        <cylinder radius="0.15" length="0.095"/>
       </geometry>
     </visual>
@@ -101,5 +101,5 @@
       <origin xyz="0 0 0" rpy="0 1.5707 1.5707"/>
       <geometry>
-        <cylinder radius="0.1" length="0.05"/>
+        <cylinder radius="0.15" length="0.095"/>
       </geometry>
     </collision>
@@ -107,5 +107,5 @@
       <origin xyz="0 0 0" rpy="0 1.5707 1.5707"/>
       <geometry>
-        <cylinder radius="0.1" length="0.05"/>
+        <cylinder radius="0.15" length="0.095"/>
       </geometry>
     </visual>
@@ -120,5 +120,5 @@
   </link>
   <joint type="continuous" name="left_wheel_hinge">
-    <origin xyz="0 0.15 0" rpy="0 0 0"/>
+    <origin xyz=".35 0.27 0" rpy="0 0 0"/>
     <!--origin xyz="0.1 0.13 0" rpy="0 1.5707 1.5707"/-->
     <child link="left_wheel"/>
@@ -129,5 +129,5 @@
   </joint>
   <joint type="continuous" name="right_wheel_hinge">
-    <origin xyz="0 -0.15 0" rpy="0 0 0"/>
+    <origin xyz=".35 -0.27 0" rpy="0 0 0"/>
     <!--origin xyz="0.1 -0.13 0" rpy="0 1.5707 1.5707"/-->
     <child link="right_wheel"/>

Commit message: works in simulation

File: src/tobor_description/urdf/tobor.xacro (robot description, xacro)
@@ -3,4 +3,6 @@
   <xacro:property name="cameraSize" value="0.05"/>
   <xacro:property name="cameraMass" value="0.1"/>
+  <xacro:property name="wheelradius" value="0.15"/>
+  <xacro:property name="wheelwidth" value="0.095"/>
   <xacro:include filename="$(find tobor_description)/urdf/tobor.gazebo" />
   <xacro:include filename="$(find tobor_description)/urdf/materials.xacro" />
@@ -9,6 +11,6 @@
     <pose>0 0 0.1 0 0 0</pose>
     <inertial>
-      <mass value="15.0"/>
-      <origin xyz="0.0 0 0.1" rpy=" 0 0 0"/>
+      <mass value="5.0"/>
+      <origin xyz="0.0 0 -0.0" rpy=" 0 0 0"/>
       <inertia
           ixx="0.1" ixy="0" ixz="0"
@@ -19,17 +21,17 @@
     <collision name='collision'>
       <geometry>
-        <box size=".78 .43 .4"/>
+        <box size=".78 .43 .2"/>
       </geometry>
     </collision>
     <visual name='chassis_visual'>
-      <origin xyz="0 0 0" rpy=" 0 0 0"/>
+      <origin xyz="0 0 -0.0" rpy=" 0 0 0"/>
       <geometry>
-        <box size=".78 .43 .4"/>
+        <box size=".78 .43 .2"/>
       </geometry>
     </visual>
     <collision name='caster_collision'>
-      <origin xyz="-0.15 0 -0.05" rpy=" 0 0 0"/>
+      <origin xyz="-0.15 0 -0.1" rpy=" 0 0 0"/>
       <geometry>
-        <sphere radius="0.05"/>
+        <sphere radius="0.0495"/>
       </geometry>
       <surface>
@@ -45,13 +47,13 @@
     </collision>
     <visual name='caster_visual'>
-      <origin xyz="-0.15 0 -0.05" rpy=" 0 0 0"/>
+      <origin xyz="-0.15 0 -0.1" rpy=" 0 0 0"/>
       <geometry>
-        <sphere radius="0.05"/>
+        <sphere radius="0.0495"/>
       </geometry>
     </visual>
     <collision name='caster_front_collision'>
-      <origin xyz="0.15 0 -0.05" rpy=" 0 0 0"/>
+      <origin xyz="0.15 0 -0.1" rpy=" 0 0 0"/>
       <geometry>
-        <sphere radius="0.05"/>
+        <sphere radius="0.0495"/>
       </geometry>
       <surface>
@@ -67,7 +69,7 @@
     </collision>
     <visual name='caster_front_visual'>
-      <origin xyz="0.15 0 -0.05" rpy=" 0 0 0"/>
+      <origin xyz="0.15 0 -0.1" rpy=" 0 0 0"/>
       <geometry>
-        <sphere radius="0.05"/>
+        <sphere radius="0.0495"/>
       </geometry>
     </visual>
@@ -78,5 +80,5 @@
       <origin xyz="0 0 0" rpy="0 1.5707 1.5707"/>
       <geometry>
-        <cylinder radius="0.15" length="0.095"/>
+         <cylinder radius="${wheelradius}" length="${wheelwidth}"/>
       </geometry>
     </collision>
@@ -84,5 +86,5 @@
       <origin xyz="0 0 0" rpy="0 1.5707 1.5707"/>
       <geometry>
-        <cylinder radius="0.15" length="0.095"/>
+        <cylinder radius="${wheelradius}" length="${wheelwidth}"/>
       </geometry>
     </visual>
@@ -101,5 +103,5 @@
       <origin xyz="0 0 0" rpy="0 1.5707 1.5707"/>
       <geometry>
-        <cylinder radius="0.15" length="0.095"/>
+        <cylinder radius="${wheelradius}" length="${wheelwidth}"/>
       </geometry>
     </collision>
@@ -107,5 +109,5 @@
       <origin xyz="0 0 0" rpy="0 1.5707 1.5707"/>
       <geometry>
-        <cylinder radius="0.15" length="0.095"/>
+        <cylinder radius="${wheelradius}" length="${wheelwidth}"/>
       </geometry>
     </visual>
@@ -120,5 +122,5 @@
   </link>
   <joint type="continuous" name="left_wheel_hinge">
-    <origin xyz=".35 0.27 0" rpy="0 0 0"/>
+    <origin xyz="0.0 0.27 0" rpy="0 0 0"/>
     <!--origin xyz="0.1 0.13 0" rpy="0 1.5707 1.5707"/-->
     <child link="left_wheel"/>
@@ -129,5 +131,5 @@
   </joint>
   <joint type="continuous" name="right_wheel_hinge">
-    <origin xyz=".35 -0.27 0" rpy="0 0 0"/>
+    <origin xyz="0.0 -0.27 0" rpy="0 0 0"/>
     <!--origin xyz="0.1 -0.13 0" rpy="0 1.5707 1.5707"/-->
     <child link="right_wheel"/>
@@ -137,4 +139,5 @@
     <joint_properties damping="1.0" friction="1.0"/>
   </joint>
+<!--
   <link name="camera">
     <collision>
@@ -164,4 +167,6 @@
     <child link="camera"/>
   </joint>
+-->
+<!--
   <joint name="hokuyo_joint" type="fixed">
     <axis xyz="0 1 0" />
@@ -170,5 +175,4 @@
     <child link="hokuyo"/>
   </joint>
-  <!-- Hokuyo Laser -->
   <link name="hokuyo">
     <collision>
@@ -190,3 +194,4 @@
     </inertial>
   </link>
+  -->
 </robot>

Commit message: moved base link

File: src/tobor_description/urdf/tobor.xacro (robot description, xacro)
@@ -3,6 +3,8 @@
   <xacro:property name="cameraSize" value="0.05"/>
   <xacro:property name="cameraMass" value="0.1"/>
-  <xacro:property name="wheelradius" value="0.15"/>
+  <xacro:property name="wheelradius" value="0.174"/>
   <xacro:property name="wheelwidth" value="0.095"/>
+  <xacro:property name="wheelDistance" value="0.54"/>
+  <xacro:property name="bodyLength" value="0.80"/>
   <xacro:include filename="$(find tobor_description)/urdf/tobor.gazebo" />
   <xacro:include filename="$(find tobor_description)/urdf/materials.xacro" />
@@ -12,12 +14,13 @@
     <inertial>
       <mass value="5.0"/>
-      <origin xyz="0.0 0 -0.0" rpy=" 0 0 0"/>
+      <origin xyz="-.2 0 0" rpy=" 0 0 0"/>
       <inertia
-          ixx="0.1" ixy="0" ixz="0"
-          iyy="0.1" iyz="0"
-          izz="0.1"
+          ixx="0.0937" ixy="0" ixz="0"
+          iyy="0.27" iyz="0"
+          izz="0.33"
       />
     </inertial>
     <collision name='collision'>
+      <origin xyz="-.2 0 0" rpy=" 0 0 0"/>
       <geometry>
         <box size=".78 .43 .2"/>
@@ -25,11 +28,11 @@
     </collision>
     <visual name='chassis_visual'>
-      <origin xyz="0 0 -0.0" rpy=" 0 0 0"/>
+      <origin xyz="-.2 0 0" rpy=" 0 0 0"/>
       <geometry>
         <box size=".78 .43 .2"/>
       </geometry>
     </visual>
-    <collision name='caster_collision'>
-      <origin xyz="-0.15 0 -0.1" rpy=" 0 0 0"/>
+    <collision name='left_caster_collision'>
+      <origin xyz="-0.50 -0.15 -0.1" rpy=" 0 0 0"/>
       <geometry>
         <sphere radius="0.0495"/>
@@ -40,4 +43,47 @@
             <mu>0</mu>
             <mu2>0</mu2>
+          </ode>
+        </friction>
+      </surface>
+    </collision>
+    <visual name='left_caster_visual'>
+      <origin xyz="-0.50 -0.15 -0.1" rpy=" 0 0 0"/>
+      <geometry>
+        <sphere radius="0.0495"/>
+      </geometry>
+    </visual>
+    <collision name='right_caster_collision'>
+        <origin xyz="-0.50 0.15 -0.1" rpy=" 0 0 0"/>
+        <geometry>
+          <sphere radius="0.0495"/>
+        </geometry>
+        <surface>
+          <friction>
+            <ode>
+              <mu>0</mu>
+              <mu2>0</mu2>
+            </ode>
+          </friction>
+        </surface>
+      </collision>
+    <visual name='right_caster_visual'>
+      <origin xyz="-0.50 0.15 -0.1" rpy=" 0 0 0"/>
+      <geometry>
+        <sphere radius="0.0495"/>
+      </geometry>
+    </visual>
+  </link>
+  <link name="left_wheel">
+    <!--origin xyz="0.1 0.13 0.1" rpy="0 1.5707 1.5707"/-->
+    <collision name="collision">
+      <origin xyz="0 0 0" rpy="0 1.5707 1.5707"/>
+      <geometry>
+         <cylinder radius="${wheelradius}" length="${wheelwidth}"/>
+      </geometry>
+      <surface>
+        <friction>
+          <ode>
+            <mu>30</mu>
+            <mu2>30</mu2>
             <slip1>1.0</slip1>
             <slip2>1.0</slip2>
@@ -46,20 +92,31 @@
       </surface>
     </collision>
-    <visual name='caster_visual'>
-      <origin xyz="-0.15 0 -0.1" rpy=" 0 0 0"/>
-      <geometry>
-        <sphere radius="0.0495"/>
-      </geometry>
-    </visual>
-    <collision name='caster_front_collision'>
-      <origin xyz="0.15 0 -0.1" rpy=" 0 0 0"/>
-      <geometry>
-        <sphere radius="0.0495"/>
+    <visual name="left_wheel_visual">
+      <origin xyz="0 0 0" rpy="0 1.5707 1.5707"/>
+      <geometry>
+        <cylinder radius="${wheelradius}" length="${wheelwidth}"/>
+      </geometry>
+    </visual>
+    <inertial>
+      <origin xyz="0 0 0" rpy="0 1.5707 1.5707"/>
+      <mass value="5"/>
+      <inertia
+        ixx=".1" ixy="0.0" ixz="0.0"
+        iyy=".1" iyz="0.0"
+        izz=".1"/>
+    </inertial>
+  </link>
+  <link name="right_wheel">
+    <!--origin xyz="0.1 -0.13 0.1" rpy="0 1.5707 1.5707"/-->
+    <collision name="collision">
+      <origin xyz="0 0 0" rpy="0 1.5707 1.5707"/>
+      <geometry>
+        <cylinder radius="${wheelradius}" length="${wheelwidth}"/>
       </geometry>
       <surface>
         <friction>
           <ode>
-            <mu>0</mu>
-            <mu2>0</mu2>
+            <mu>30</mu>
+            <mu2>30</mu2>
             <slip1>1.0</slip1>
             <slip2>1.0</slip2>
@@ -68,20 +125,5 @@
       </surface>
     </collision>
-    <visual name='caster_front_visual'>
-      <origin xyz="0.15 0 -0.1" rpy=" 0 0 0"/>
-      <geometry>
-        <sphere radius="0.0495"/>
-      </geometry>
-    </visual>
-  </link>
-  <link name="left_wheel">
-    <!--origin xyz="0.1 0.13 0.1" rpy="0 1.5707 1.5707"/-->
-    <collision name="collision">
-      <origin xyz="0 0 0" rpy="0 1.5707 1.5707"/>
-      <geometry>
-         <cylinder radius="${wheelradius}" length="${wheelwidth}"/>
-      </geometry>
-    </collision>
-    <visual name="left_wheel_visual">
+    <visual name="right_wheel_visual">
       <origin xyz="0 0 0" rpy="0 1.5707 1.5707"/>
       <geometry>
@@ -98,27 +140,4 @@
     </inertial>
   </link>
-  <link name="right_wheel">
-    <!--origin xyz="0.1 -0.13 0.1" rpy="0 1.5707 1.5707"/-->
-    <collision name="collision">
-      <origin xyz="0 0 0" rpy="0 1.5707 1.5707"/>
-      <geometry>
-        <cylinder radius="${wheelradius}" length="${wheelwidth}"/>
-      </geometry>
-    </collision>
-    <visual name="right_wheel_visual">
-      <origin xyz="0 0 0" rpy="0 1.5707 1.5707"/>
-      <geometry>
-        <cylinder radius="${wheelradius}" length="${wheelwidth}"/>
-      </geometry>
-    </visual>
-    <inertial>
-      <origin xyz="0 0 0" rpy="0 1.5707 1.5707"/>
-      <mass value="5"/>
-      <inertia
-        ixx=".1" ixy="0.0" ixz="0.0"
-        iyy=".1" iyz="0.0"
-        izz=".1"/>
-    </inertial>
-  </link>
   <joint type="continuous" name="left_wheel_hinge">
     <origin xyz="0.0 0.27 0" rpy="0 0 0"/>
@@ -139,4 +158,21 @@
     <joint_properties damping="1.0" friction="1.0"/>
   </joint>
+<!--
+  <link name="baselink">
+    <collision>
+      <origin xyz="0 0 0" rpy=" 0 0 0"/>
+      <geometry>
+        <box size=".2 .38 .2"/>
+      </geometry>
+    </collision>
+    <visual>
+      <origin xyz="0 0 -0.0" rpy=" 0 0 0"/>
+      <geometry>
+        <box size=".2 .38 .2"/>
+      </geometry>
+      <material name="black"/>
+    </visual>
+  </link>
+  -->
 <!--
   <link name="camera">

Commit message: added body+inertia

File: src/tobor_description/urdf/tobor.xacro (robot description, xacro)
@@ -7,4 +7,5 @@
   <xacro:property name="wheelDistance" value="0.54"/>
   <xacro:property name="bodyLength" value="0.80"/>
+  <xacro:property name="casterRadius" value="0.05"/>
   <xacro:include filename="$(find tobor_description)/urdf/tobor.gazebo" />
   <xacro:include filename="$(find tobor_description)/urdf/materials.xacro" />
@@ -12,17 +13,8 @@
   <link name='base_link'>
     <pose>0 0 0.1 0 0 0</pose>
-    <inertial>
-      <mass value="5.0"/>
-      <origin xyz="-.2 0 0" rpy=" 0 0 0"/>
-      <inertia
-          ixx="0.0937" ixy="0" ixz="0"
-          iyy="0.27" iyz="0"
-          izz="0.33"
-      />
-    </inertial>
     <collision name='collision'>
       <origin xyz="-.2 0 0" rpy=" 0 0 0"/>
       <geometry>
-        <box size=".78 .43 .2"/>
+        <box size=".78 .43 .05"/>
       </geometry>
     </collision>
@@ -30,11 +22,11 @@
       <origin xyz="-.2 0 0" rpy=" 0 0 0"/>
       <geometry>
-        <box size=".78 .43 .2"/>
+        <box size=".78 .43 .05"/>
       </geometry>
     </visual>
     <collision name='left_caster_collision'>
-      <origin xyz="-0.50 -0.15 -0.1" rpy=" 0 0 0"/>
-      <geometry>
-        <sphere radius="0.0495"/>
+      <origin xyz="-0.50 -0.15 -${wheelradius-casterRadius}" rpy=" 0 0 0"/>
+      <geometry>
+        <sphere radius="${casterRadius}"/>
       </geometry>
       <surface>
@@ -48,13 +40,13 @@
     </collision>
     <visual name='left_caster_visual'>
-      <origin xyz="-0.50 -0.15 -0.1" rpy=" 0 0 0"/>
-      <geometry>
-        <sphere radius="0.0495"/>
+      <origin xyz="-0.50 -0.15 -0.12" rpy=" 0 0 0"/>
+      <geometry>
+        <sphere radius="${casterRadius}"/>
       </geometry>
     </visual>
     <collision name='right_caster_collision'>
-        <origin xyz="-0.50 0.15 -0.1" rpy=" 0 0 0"/>
+        <origin xyz="-0.50 0.15 -0.12" rpy=" 0 0 0"/>
         <geometry>
-          <sphere radius="0.0495"/>
+          <sphere radius="${casterRadius}"/>
         </geometry>
         <surface>
@@ -68,7 +60,7 @@
       </collision>
     <visual name='right_caster_visual'>
-      <origin xyz="-0.50 0.15 -0.1" rpy=" 0 0 0"/>
-      <geometry>
-        <sphere radius="0.0495"/>
+      <origin xyz="-0.50 0.15 -0.12" rpy=" 0 0 0"/>
+      <geometry>
+        <sphere radius="${casterRadius}"/>
       </geometry>
     </visual>
@@ -158,4 +150,36 @@
     <joint_properties damping="1.0" friction="1.0"/>
   </joint>
+  <link name="body">
+    <!--origin xyz="0.1 -0.13 0.1" rpy="0 1.5707 1.5707"/-->
+    <collision name="collision">
+      <origin xyz="-.2 0 0.1" rpy=" 0 0 0"/>
+      <geometry>
+        <box size=".78 .43 .35"/>
+      </geometry>
+    </collision>
+    <visual name="right_wheel_visual">
+      <origin xyz="-.2 0 0.3" rpy=" 0 0 0"/>
+      <geometry>
+        <box size=".78 .43 .35"/>
+      </geometry>
+      <material name="yellow"/>
+    </visual>
+   <inertial>
+      <mass value="5.0"/>
+      <origin xyz="-.2 0 0" rpy=" 0 0 0"/>
+      <inertia
+          ixx="0.0937" ixy="0" ixz="0"
+          iyy="0.27" iyz="0"
+          izz="0.33"
+      />
+    </inertial>
+  </link>
+  <joint type="fixed" name="body_hinge">
+    <origin xyz="0 0 0" rpy="0 0 0"/>
+    <!--origin xyz="0.1 -0.13 0" rpy="0 1.5707 1.5707"/-->
+    <child link="body"/>
+    <parent link="base_link"/>
+    <axis xyz="0 0 0" rpy="0 0 0"/>
+  </joint>
 <!--
   <link name="baselink">

Commit message: enabled mapping again

File: src/tobor_description/urdf/tobor.xacro (robot description, xacro)
@@ -182,22 +182,4 @@
     <axis xyz="0 0 0" rpy="0 0 0"/>
   </joint>
-<!--
-  <link name="baselink">
-    <collision>
-      <origin xyz="0 0 0" rpy=" 0 0 0"/>
-      <geometry>
-        <box size=".2 .38 .2"/>
-      </geometry>
-    </collision>
-    <visual>
-      <origin xyz="0 0 -0.0" rpy=" 0 0 0"/>
-      <geometry>
-        <box size=".2 .38 .2"/>
-      </geometry>
-      <material name="black"/>
-    </visual>
-  </link>
-  -->
-<!--
   <link name="camera">
     <collision>
@@ -223,13 +205,11 @@
   <joint name="camera_joint" type="fixed">
     <axis xyz="0 1 0" />
-    <origin xyz=".2 0 0" rpy="0 0 0"/>
+    <origin xyz=".2 0 .2" rpy="0 0 0"/>
     <parent link="base_link"/>
     <child link="camera"/>
   </joint>
--->
-<!--
   <joint name="hokuyo_joint" type="fixed">
     <axis xyz="0 1 0" />
-    <origin xyz=".15 0 .1" rpy="0 0 0"/>
+    <origin xyz=".2 0 .3" rpy="0 0 0"/>
     <parent link="base_link"/>
     <child link="hokuyo"/>
@@ -254,4 +234,3 @@
     </inertial>
   </link>
-  -->
 </robot>
